File: pcb/OpenScrewCounter/OpenScrewCounter.kicad_sch (KiCad schematic)
At the start: 24 parts

Commit message: pcb update
Parts:
- removed D? (x4): LED, LED_THT:LED_D5.0mm, symbol Device:LED
- removed J?: IN, TerminalBlock_Phoenix:TerminalBlock_Phoenix_MKDS-1,5-2-5.08_1x02_P5.08mm_Horizontal, symbol Connector:Screw_Terminal_01x02
- removed JP?: J_BUZZ, Jumper:SolderJumper-2_P1.3mm_Open_Pad1.0x1.5mm, symbol Jumper:SolderJumper_2_Open
- removed R?: 10k, Resistor_SMD:R_0603_1608Metric_Pad0.98x0.95mm_HandSolder, symbol Device:R
- removed R? (x4): 330, Resistor_SMD:R_1206_3216Metric_Pad1.30x1.75mm_HandSolder, symbol Device:R
- removed U? (x3): tact_switch, casual_components:tact_switch, symbol casual_components:tact_switch
- added J1, J3, J4: Sensor, Connector_PinHeader_2.54mm:PinHeader_1x03_P2.54mm_Vertical, symbol Connector:Conn_01x03_Male
- added R1, R2, R3, R4, R5, R6, R7, R8: 330, Resistor_SMD:R_1206_3216Metric_Pad1.30x1.75mm_HandSolder, symbol Device:R
- added SW1, SW2, SW3: SW_Push, Button_Switch_THT:SW_PUSH_6mm_H7.3mm, symbol Switch:SW_Push
- J5: renamed from J?; footprint (none) -> Connector_BarrelJack:BarrelJack_Horizontal
- gave numbers to parts that had none: 9
Connections:
- net +12V: now also J5.1; no longer J2.1 (Pin_1)
- net +3V3: now also J1.1 (Pin_1), J3.1 (Pin_1), J4.1 (Pin_1), SW1.1, SW2.1, SW3.1
- net +5V: now also J2.1 (Pin_1)
- net BUTTON1: now also U2.5 (GP3), SW3.2
- net BUTTON2: now also U2.11 (GP8), SW2.2
- net BUTTON3: now also U2.12 (GP9), SW1.2
- net BUZZER: now also BZ1.1 (-), U2.4 (GP2)
- net GND: now also J5.2, J1.2 (Pin_2), J3.2 (Pin_2), J4.2 (Pin_2)
- net MOTOR: now also U2.21 (GP16); no longer U2.20 (GP15)
- net at U1.1 (e): now also R5.2
- net at U1.10 (f): now also R6.2
- net at U1.11 (a): now also R1.2
- net DIG1: now reaches U1.12 (CA1)
- net DIG1: now also U2.24 (GP18)
- net at U1.2 (d): now also R4.2
- net at U1.3 (DPX): now also R8.2
- net at U1.4 (c): now also R3.2
- net at U1.5 (g): now also R7.2
- net at U1.7 (b): now also R2.2
- net DIG3: now reaches U1.8 (CA3)
- net DIG3: now also U2.29 (GP22)
- net DIG2: now reaches U1.9 (CA2)
- net DIG2: now also U2.27 (GP21)
- net SENSOR1: now reaches U2.10 (GP7)
- net SENSOR1: now also J3.3 (Pin_3)
- net DIS_B: now reaches U2.14 (GP10)
- net DIS_B: now also R2.1
- net DIS_G: now reaches U2.15 (GP11)
- net DIS_G: now also R7.1
- net DIS_C: now reaches U2.16 (GP12)
- net DIS_C: now also R3.1
- net DIS_DP: now reaches U2.17 (GP13)
- net DIS_DP: now also R8.1
- net DIS_D: now reaches U2.19 (GP14)
- net DIS_D: now also R4.1
- net DIS_A: now reaches U2.25 (GP19)
- net DIS_A: now also R1.1
- net DIS_F: now reaches U2.26 (GP20)
- net DIS_F: now also R6.1
- net SENSOR3: now reaches U2.7 (GP5)
- net SENSOR3: now also J1.3 (Pin_3)
- net SENSOR2: now reaches U2.9 (GP6)
- net SENSOR2: now also J4.3 (Pin_3)
- new net DIS_E: R5.1, U2.20 (GP15)
Other:
- moved on the sheet: U1
