File: pcb/OpenScrewCounter/OpenScrewCounter.kicad_pcb (KiCad board)
At the start: 2 copper layers, 54.6 x 85.1 mm, 28 parts, among them J2 P1, J5 Barrel_Jack_MountingPin, Q1 IRFZ44N, SW1 SW_Push, SW2 SW_Push, SW3 SW_Push, U1 CA56-12EWA, U2 pi pico, U3 L7805

Commit message: pcb gcode and fix
Routing:
- net GND: track 58.7 -> 87.7 mm, vias 0 -> 1
Changed lines of the file:
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@@
   (segment (start 122.081031 118.436031) (end 122.081031 114.507101) (width 0.762) (layer "B.Cu") (net 1))
   (segment (start 123.8 120.155) (end 122.081031 118.436031) (width 0.762) (layer "B.Cu") (net 1))
+  (segment (start 99.06 85.09) (end 99.06 97.79) (width 0.762) (layer "F.Cu") (net 2))
   (segment (start 113.03 111.76) (end 116.133791 108.656209) (width 0.762) (layer "F.Cu") (net 2))
   (segment (start 113.03 114.3) (end 113.03 111.76) (width 0.762) (layer "F.Cu") (net 2))
+  (segment (start 85.85 77.57) (end 91.54 77.57) (width 0.762) (layer "F.Cu") (net 2))
+  (segment (start 91.54 77.57) (end 99.06 85.09) (width 0.762) (layer "F.Cu") (net 2))
   (segment (start 116.133791 108.656209) (end 119.069041 108.656209) (width 0.762) (layer "F.Cu") (net 2))
+  (via (at 99.06 97.79) (size 0.8) (drill 0.4) (layers "F.Cu" "B.Cu") (net 2))
   (segment (start 106.695 118.125) (end 108.142163 119.572163) (width 0.508) (layer "B.Cu") (net 2))
   (segment (start 125.962959 107.717041) (end 131.847041 107.717041) (width 0.762) (layer "B.Cu") (net 2))
